Commit message: Comment details

File: Aula12/p_rsiopa_description/urdf/p_rsiopa.gazebo.macro.xacro (robot description, xacro)
@@ -1,9 +1,11 @@
 <?xml version="1.0"?>
 <robot name="p_rsiopa" xmlns:xacro="http://ros.org/wiki/xacro">
-  <xacro:arg name="laser_visual"  default="false"/>
-  <xacro:arg name="camera_visual" default="false"/>
-  <xacro:arg name="imu_visual"    default="false"/>
+  <xacro:macro name="gazebo_macro" params="player_color laser_visual camera_visual imu_visual">
+<!--  <xacro:macro name="gazebo_macro" params="player_color">-->
+<!--  <xacro:arg name="laser_visual"  default="false"/>-->
+<!--  <xacro:arg name="camera_visual" default="false"/>-->
+<!--  <xacro:arg name="imu_visual"    default="false"/>-->
   <gazebo reference="base_link">
-    <material>Gazebo/DarkGrey</material>
+    <material>Gazebo/${player_color}</material>
   </gazebo>
   <gazebo reference="wheel_left_link">
@@ -15,5 +17,6 @@
     <maxVel>0.1</maxVel>
     <fdir1>1 0 0</fdir1>
-    <material>Gazebo/Orange</material>
+    <material>Gazebo/FlatBlack</material>
+<!--    <material>Gazebo/Blue</material>-->
   </gazebo>
   <gazebo reference="wheel_right_link">
@@ -25,5 +28,6 @@
     <maxVel>0.1</maxVel>
     <fdir1>1 0 0</fdir1>
-    <material>Gazebo/Orange</material>
+    <material>Gazebo/FlatBlack</material>
+<!--    <material>Gazebo/Blue</material>-->
   </gazebo>
   <gazebo reference="caster_back_right_link">
@@ -34,5 +38,5 @@
     <minDepth>0.001</minDepth>
     <maxVel>1.0</maxVel>
-    <material>Gazebo/Orange</material>
+    <material>Gazebo/FlatBlack</material>
   </gazebo>
   <gazebo reference="caster_back_left_link">
@@ -43,12 +47,12 @@
     <minDepth>0.001</minDepth>
     <maxVel>1.0</maxVel>
-    <material>Gazebo/Orange</material>
+    <material>Gazebo/FlatBlack</material>
   </gazebo>
   <gazebo reference="imu_link">
     <sensor type="imu" name="imu">
       <always_on>true</always_on>
-      <visualize>$(arg imu_visual)</visualize>
+      <visualize>${imu_visual}</visualize>
     </sensor>
-    <material>Gazebo/Orange</material>
+    <material>Gazebo/Grey</material>
   </gazebo>
   <gazebo>
@@ -103,8 +107,8 @@
   </gazebo>
   <gazebo reference="base_scan">
-    <material>Gazebo/Orange</material>
+    <material>Gazebo/FlatBlack</material>
     <sensor type="ray" name="lds_lfcd_sensor">
       <pose>0 0 0 0 0 0</pose>
-      <visualize>$(arg laser_visual)</visualize>
+      <visualize>${laser_visual}</visualize>
       <update_rate>5</update_rate>
       <ray>
@@ -138,5 +142,5 @@
     <sensor type="camera" name="Pi Camera">
       <always_on>true</always_on>
-      <visualize>$(arg camera_visual)</visualize>
+      <visualize>${camera_visual}</visualize>
       <camera>
           <horizontal_fov>1.085595</horizontal_fov>
@@ -167,3 +171,4 @@
     </sensor>
   </gazebo>
+  </xacro:macro>
 </robot>

File: Aula12/p_rsiopa_description/urdf/p_rsiopa.urdf.xacro (robot description, xacro)
@@ -1,6 +1,18 @@
 <?xml version="1.0" ?>
-<robot name="turtlebot3" xmlns:xacro="http://ros.org/wiki/xacro">
+<robot name="p_rsiopa" xmlns:xacro="http://ros.org/wiki/xacro">
   <xacro:include filename="$(find turtlebot3_description)/urdf/common_properties.xacro"/>
-  <xacro:include filename="$(find p_rsiopa_description)/urdf/p_rsiopa.gazebo.xacro"/>
+<!--  <xacro:include filename="$(find p_rsiopa_description)/urdf/p_rsiopa.gazebo.xacro"/>-->
+  <!--Args are local, properties are global, so we copy the values of the arguments to the properties-->
+  <xacro:arg name="player_name" default="p_rsiopa" />
+  <xacro:arg name="player_color" default="Orange" />
+  <!-- e.g. Red, Orange. Must exist in Gazebo/Colors and be defined in properties.xacro.-->
+  <!--Properties are global so they can be viewed from inside the included xacros-->
+  <!--  args are used with $(arg arg_name), properties are used as ${property_name}-->
+  <xacro:property name="player_name" value="$(arg player_name)"/>
+  <xacro:property name="player_color" value="$(arg player_color)"/>
+  <!-- Include other files-->
+  <xacro:include filename="$(find p_rsiopa_description)/urdf/p_rsiopa.gazebo.macro.xacro"/>
+  <xacro:gazebo_macro player_color="${player_color}" laser_visual="false" camera_visual="false" imu_visual="false"/>
+<!--  <xacro:gazebo_macro player_color="${player_color}" />-->
   <link name="base_footprint"/>
   <joint name="base_joint" type="fixed">
